Commit message: Update README.md, params and RViz bug

File: description/robot_core.xacro (robot description, xacro)
@@ -10,4 +10,7 @@
     <material name="blue">
         <color rgba="0.2 0.2 1 1"/>
+    </material>
+    <material name="grey">
+        <color rgba="0.5 0.5 0.5 1"/>
     </material>
     <!-- BASE LINK -->
@@ -34,5 +37,5 @@
                 <cylinder radius="0.105" length="0.062"/>
             </geometry>
-            <material name="white"/>
+            <material name="grey"/>
         </visual>
         <collision>
@@ -47,5 +50,5 @@
     </link>
     <gazebo reference="chassis">
-        <material>Gazebo/White</material>
+        <material>Gazebo/Gray</material>
     </gazebo>
     <!-- LEFT WHEEL LINK -->

Commit message: Fix wheel rolling and README typo

File: description/robot_core.xacro (robot description, xacro)
@@ -45,6 +45,6 @@
             </geometry>
         </collision>
-        <xacro:inertial_cylinder mass="10" length="0.062" radius="0.105">
-            <origin xyz="0.105 0 0.06025" rpy="0 0 0"/>
+        <xacro:inertial_cylinder mass="2" length="0.062" radius="0.105">
+            <origin xyz="0.105 0 0.007" rpy="0 0 0"/>
         </xacro:inertial_cylinder>
     </link>
@@ -72,5 +72,5 @@
             </geometry>
         </collision>
-        <xacro:inertial_cylinder mass="0.1" length="0.01" radius="0.02075">
+        <xacro:inertial_cylinder mass="5" length="0.01" radius="0.02075">
             <origin xyz="0 0 0" rpy="0 0 0"/>
         </xacro:inertial_cylinder>
@@ -99,5 +99,5 @@
             </geometry>
         </collision>
-        <xacro:inertial_cylinder mass="0.1" length="0.01" radius="0.02075">
+        <xacro:inertial_cylinder mass="5" length="0.01" radius="0.02075">
             <origin xyz="0 0 0" rpy="0 0 0"/>
         </xacro:inertial_cylinder>
@@ -124,5 +124,5 @@
             </geometry>
         </collision>
-        <xacro:inertial_sphere mass="0.1" radius="0.02">
+        <xacro:inertial_sphere mass="5" radius="0.02">
             <origin xyz="0 0 0" rpy="0 0 0"/>
         </xacro:inertial_sphere>
