Commit message: Reset params

File: description/camera.xacro (robot description, xacro)
@@ -17,5 +17,5 @@
         <parent link="chassis"/>
         <child link="camera_link"/>
-        <origin xyz="0.255 0 0.05" rpy="0 0 0"/>
+        <origin xyz="0.26 0 0.05" rpy="0 0 0"/>
     </joint>
    <link name="camera_link"></link>

Commit message: Improving launch files

File: description/camera.xacro (robot description, xacro)
@@ -9,6 +9,7 @@
         <visual>
             <geometry>
-                <!--<mesh filename="package://mogbe/meshes/RasPi-Camera-v1.obj" scale="0.001 0.001 0.001"/>-->
-                <mesh filename="file://$(find mogbe)/meshes/RasPi-Camera-v1.obj" scale="0.001 0.001 0.001"/>
+                <!--<mesh filename="package://mogbe/meshes/RasPi-Camera-v1.obj" scale="0.001 0.001 0.001"/> SÓ FUNCIONA COM RVIZ -->
+                <!--<mesh filename="file://$(find mogbe)/meshes/RasPi-Camera-v1.obj" scale="0.001 0.001 0.001"/> FUNCIONA COM GAZEBO E RVIZ SOMENTE EM SIMULAÇÃO -->
+                <mesh filename="file:///home/dev/dev_ws/src/mogbe/meshes/RasPi-Camera-v1.obj" scale="0.001 0.001 0.001"/> <!-- FUNCIONA GAZEBO E RVIZ, SIM E REAL -->
             </geometry>
         </visual>

File: description/lidar.xacro (robot description, xacro)
@@ -10,5 +10,7 @@
             <geometry>
                 <!--<cylinder radius="0.05" length="0.04"/>-->
-                <mesh filename="file://$(find mogbe)/meshes/LD19-v1.obj" scale="0.001 0.001 0.001"/>
+                <!--<mesh filename="file://$(find mogbe)/meshes/LD19-v1.obj" scale="0.001 0.001 0.001"/> SÓ FUNCIONA COM RVIZ -->
+                <!-- <mesh filename="file://$(find mogbe)/meshes/LD19-v1.obj" scale="0.001 0.001 0.001"/> FUNCIONA COM GAZEBO E RVIZ SOMENTE EM SIMULAÇÃO -->
+                <mesh filename="file:///home/dev/dev_ws/src/mogbe/meshes/LD19-v1.obj" scale="0.001 0.001 0.001"/> <!-- FUNCIONA GAZEBO E RVIZ, SIM E REAL -->
             </geometry>
             <!--<material name="blue"/>-->

Commit message: Update README

File: description/camera.xacro (robot description, xacro)
@@ -11,5 +11,5 @@
                 <!--<mesh filename="package://mogbe/meshes/RasPi-Camera-v1.obj" scale="0.001 0.001 0.001"/> SÓ FUNCIONA COM RVIZ -->
                 <!--<mesh filename="file://$(find mogbe)/meshes/RasPi-Camera-v1.obj" scale="0.001 0.001 0.001"/> FUNCIONA COM GAZEBO E RVIZ SOMENTE EM SIMULAÇÃO -->
-                <mesh filename="file:///home/dev/dev_ws/src/mogbe/meshes/RasPi-Camera-v1.obj" scale="0.001 0.001 0.001"/> <!-- FUNCIONA GAZEBO E RVIZ, SIM E REAL -->
+                <mesh filename="file:///home/dev/mogbe_ws/src/mogbe/meshes/RasPi-Camera-v1.obj" scale="0.001 0.001 0.001"/> <!-- FUNCIONA GAZEBO E RVIZ, SIM E REAL -->
             </geometry>
         </visual>

File: description/lidar.xacro (robot description, xacro)
@@ -12,5 +12,5 @@
                 <!--<mesh filename="file://$(find mogbe)/meshes/LD19-v1.obj" scale="0.001 0.001 0.001"/> SÓ FUNCIONA COM RVIZ -->
                 <!-- <mesh filename="file://$(find mogbe)/meshes/LD19-v1.obj" scale="0.001 0.001 0.001"/> FUNCIONA COM GAZEBO E RVIZ SOMENTE EM SIMULAÇÃO -->
-                <mesh filename="file:///home/dev/dev_ws/src/mogbe/meshes/LD19-v1.obj" scale="0.001 0.001 0.001"/> <!-- FUNCIONA GAZEBO E RVIZ, SIM E REAL -->
+                <mesh filename="file:///home/dev/mogbe_ws/src/mogbe/meshes/LD19-v1.obj" scale="0.001 0.001 0.001"/> <!-- FUNCIONA GAZEBO E RVIZ, SIMULAÇÃO E REAL -->
             </geometry>
             <!--<material name="blue"/>-->

Commit message: Fix absolute path dependencies + deprecated usage + typo

File: description/camera.xacro (robot description, xacro)
@@ -9,7 +9,10 @@
         <visual>
             <geometry>
-                <!--<mesh filename="package://mogbe/meshes/RasPi-Camera-v1.obj" scale="0.001 0.001 0.001"/> SÓ FUNCIONA COM RVIZ -->
-                <!--<mesh filename="file://$(find mogbe)/meshes/RasPi-Camera-v1.obj" scale="0.001 0.001 0.001"/> FUNCIONA COM GAZEBO E RVIZ SOMENTE EM SIMULAÇÃO -->
-                <mesh filename="file:///home/dev/mogbe_ws/src/mogbe/meshes/RasPi-Camera-v1.obj" scale="0.001 0.001 0.001"/> <!-- FUNCIONA GAZEBO E RVIZ, SIM E REAL -->
+                <xacro:if value="$(arg sim_mode)">
+                    <mesh filename="file://$(find mogbe)/meshes/RasPi-Camera-v1.obj" scale="0.001 0.001 0.001"/>
+                </xacro:if>
+                <xacro:unless value="$(arg sim_mode)">
+                    <mesh filename="package://mogbe/meshes/RasPi-Camera-v1.obj" scale="0.001 0.001 0.001"/>
+                </xacro:unless>
             </geometry>
         </visual>

File: description/lidar.xacro (robot description, xacro)
@@ -9,10 +9,11 @@
         <visual>
             <geometry>
-                <!--<cylinder radius="0.05" length="0.04"/>-->
-                <!--<mesh filename="file://$(find mogbe)/meshes/LD19-v1.obj" scale="0.001 0.001 0.001"/> SÓ FUNCIONA COM RVIZ -->
-                <!-- <mesh filename="file://$(find mogbe)/meshes/LD19-v1.obj" scale="0.001 0.001 0.001"/> FUNCIONA COM GAZEBO E RVIZ SOMENTE EM SIMULAÇÃO -->
-                <mesh filename="file:///home/dev/mogbe_ws/src/mogbe/meshes/LD19-v1.obj" scale="0.001 0.001 0.001"/> <!-- FUNCIONA GAZEBO E RVIZ, SIMULAÇÃO E REAL -->
+                <xacro:if value="$(arg sim_mode)">
+                    <mesh filename="file://$(find mogbe)/meshes/LD19-v1.obj" scale="0.001 0.001 0.001"/>
+                </xacro:if>
+                <xacro:unless value="$(arg sim_mode)">
+                    <mesh filename="package://mogbe/meshes/LD19-v1.obj" scale="0.001 0.001 0.001"/>
+                </xacro:unless>
             </geometry>
-            <!--<material name="blue"/>-->
         </visual>
         <collision>
@@ -53,5 +54,5 @@
             <plugin name="laser_controller" filename="libgazebo_ros_ray_sensor.so">
                 <ros>
-                    <argument>~/out:=scan</argument>
+                    <remapping>~/out:=scan</remapping>
                 </ros>
                 <output_type>sensor_msgs/LaserScan</output_type>
